File: Vanguard_V2/IO.kicad_sch (KiCad schematic)
At the start: 22 parts, among them J2 Conn_01x05_Pin, J3 MEM2067-02-180-00-A, J4 Conn_01x04_Pin, J5 Conn_01x02_Pin, J6 Conn_01x02_Pin, J8 USB_B_Micro, SW1 SW_Push, SW2 SW_Push, U3 USBLC6-2P6

Commit message: V2 Board Ready
Parts:
- removed J6: Conn_01x02_Pin, Connector_PinHeader_2.54mm:PinHeader_1x02_P2.54mm_Vertical, symbol Connector:Conn_01x02_Pin
- removed R10: 10k, Resistor_SMD:R_0402_1005Metric, symbol Device:R
