File: Vanguard_V2/Power.kicad_sch (KiCad schematic)
At the start: 17 parts, among them IC1 ST1L05CPU33R, J1 Conn_01x02_Pin, U2 LD1117S50TR_SOT223

Commit message: Added ejection charges
Parts:
- C7: footprint Capacitor_SMD:C_0603_1608Metric -> Capacitor_SMD:C_0402_1005Metric
Changed lines of the file:
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@@
 			)
 		)
-		(property "Footprint" "Capacitor_SMD:C_0603_1608Metric"
+		(property "Footprint" "Capacitor_SMD:C_0402_1005Metric"
 			(at 32.7152 93.98 0)
 			(effects

Commit message: Fixed sensors
Parts:
- added D7: CDBU0520, Resistor_SMD:R_0402_1005Metric, symbol PartDB:CDBU0520
Connections:
- net VIN: now also D7.2 (A); no longer C7.1, U2.3 (VI)
- new net VBATT: C7.1, D7.1 (K), U2.3 (VI)
